File: RF.kicad_sch (KiCad schematic)
At the start: 0 parts

Commit message: added rudimentary RF matching network
Parts:
- added AE1: ANT_00001, symbol mic_patch_parts:ANT_00001
- added C25: C_00008_RF, symbol mic_patch_parts:C_00008_RF
- added C26: C_00007_RF, symbol mic_patch_parts:C_00007_RF
- added C27: C_00009_RF, symbol mic_patch_parts:C_00009_RF
- added L4: L_00003_RF, symbol mic_patch_parts:L_00003_RF
- added L5: L_00004_RF, symbol mic_patch_parts:L_00004_RF
- added L6: L_00005_RF, symbol mic_patch_parts:L_00005_RF_1
Connections:
- new net: C25.1, C27.2, L4.2
- new net: C27.1, L5.1, L6.1
- new net: AE1.1 (FEED), L5.2
- new net GND: C25.2, C26.2, L6.2
- new net RF_ANT: C26.1, L4.1
- no-connect marks 0 -> 1
Other:
- note added: "50ohm impedance line"
- note added: "Check package for extra cap...."
- note added: "NRF5340 Radio Matching network"

Commit message: tided up
Other:
- note added: "50ohm impedance"
- note added: "Antenna Impedance matching network"
- note removed: "50ohm impedance line"
Changed lines of the file:
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@@
+		)
+	)
+	(text "Antenna Impedance matching network"
+		(exclude_from_sim no)
+		(at 146.812 72.39 0)
+		(effects
+			(font
+				(size 1.27 1.27)
+			)
 		)
 	)
@@
 		)
 	)
-	(text "50ohm impedance line"
+	(text "50ohm impedance"
 		(exclude_from_sim no)
-		(at 117.856 85.598 0)
+		(at 117.602 81.534 0)
 		(effects
 			(font
