File: MCU.kicad_sch (KiCad schematic)
At the start: 13 parts, among them J1 Conn_ARM_SWD_TagConnect_TC203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, SW1 SW_000001, SW2 SW_000001, U1 NORA-B106-00B, Y1 CLK_0003

Commit message: routed every component, added GPIO breakouts
Parts:
- added TP5: GPIO Breakout P1.06, TestPoint:TestPoint_Pad_D1.0mm, symbol Connector:TestPoint
- added TP6: GPIO Breakout P0.24, TestPoint:TestPoint_Pad_D1.0mm, symbol Connector:TestPoint
Connections:
- net at U1.G1 (P1.06): now also TP5.1
- net at U1.H1 (P0.24): now also TP6.1
- no-connect marks 35 -> 33
Changed lines of the file:
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@@
-	)
-	(no_connect
-		(at 142.24 93.98)
-	)
-	(no_connect
-		(at 86.36 139.7)
 	)
 	(no_connect
@@
 	(wire
 		(pts
+			(xy 142.24 93.98) (xy 166.37 93.98)
+		)
+		(stroke
+			(width 0)
+			(type default)
+		)
+	)
+	(wire
+		(pts
 			(xy 133.35 170.18) (xy 135.89 170.18)
 		)
@@
 	(wire
 		(pts
+			(xy 86.36 139.7) (xy 71.12 139.7)
+		)
+		(stroke
+			(width 0)
+			(type default)
+		)
+	)
+	(wire
+		(pts
 			(xy 96.52 170.18) (xy 99.06 170.18)
 		)
@@
 	(wire
 		(pts
-			(xy 142.24 91.44) (xy 147.32 91.44)
+			(xy 71.12 139.7) (xy 69.85 138.43)
+		)
+		(stroke
+			(width 0)
+			(type default)
+		)
+	)
+	(wire
+		(pts
+			(xy 146.05 86.36) (xy 147.32 86.36)
 		)
 		(stroke
@@
 	(wire
 		(pts
+			(xy 146.05 91.44) (xy 142.24 91.44)
+		)
+		(stroke
+			(width 0)
+			(type default)
+		)
+	)
+	(wire
+		(pts
 			(xy 180.34 64.77) (xy 186.69 64.77)
 		)
@@
 		(pts
 			(xy 147.32 68.58) (xy 147.32 71.12)
+		)
+		(stroke
+			(width 0)
+			(type default)
+		)
+	)
+	(wire
+		(pts
+			(xy 146.05 86.36) (xy 146.05 91.44)
+		)
+		(stroke
+			(width 0)
+			(type default)
+		)
+	)
+	(wire
+		(pts
+			(xy 166.37 93.98) (xy 167.64 92.71)
 		)
 		(stroke
@@
 	(global_label "NPM MODE"
 		(shape input)
-		(at 147.32 91.44 0)
+		(at 147.32 86.36 0)
 		(fields_autoplaced yes)
 		(effects
@@
 		)
 		(property "Intersheetrefs" "${INTERSHEET_REFS}"
-			(at 160.5256 91.44 0)
+			(at 160.5256 86.36 0)
 			(effects
 				(font
@@
 					(unit 1)
 				)
+			)
+		)
+	)
+	(symbol
+		(lib_id "Connector:TestPoint")
+		(at 167.64 92.71 0)
+		(unit 1)
+		(exclude_from_sim no)
+		(in_bom yes)
+		(on_board yes)
+		(dnp no)
+		(property "Reference" "TP5"
+			(at 165.862 87.63 0)
+			(effects
+				(font
+					(size 1.27 1.27)
+				)
+				(justify left)
+			)
+		)
+		(property "Value" "GPIO Breakout P1.06"
+			(at 162.306 84.836 0)
+			(effects
+				(font
+					(size 1.27 1.27)
+				)
+				(justify left)
+			)
+		)
+		(property "Footprint" "TestPoint:TestPoint_Pad_D1.0mm"
+			(at 172.72 92.71 0)
+			(effects
+				(font
+					(size 1.27 1.27)
+				)
+				(hide yes)
+			)
+		)
+		(property "Datasheet" "~"
+			(at 172.72 92.71 0)
+			(effects
+				(font
+					(size 1.27 1.27)
+				)
+				(hide yes)
+			)
+		)
+		(property "Description" "test point"
+			(at 167.64 92.71 0)
+			(effects
+				(font
+					(size 1.27 1.27)
+				)
+				(hide yes)
+			)
+		)
+		(pin "1"
+		)
+		(instances
+			(project "mic_patch_v1"
+				(path "/5448a297-4261-40a5-8009-47199bfe22cb/1e8f7a85-c9d9-4dea-908a-5a79456d7ca4"
+					(reference "TP5")
+					(unit 1)
+				)
+			)
+		)
+	)
+	(symbol
+		(lib_id "Connector:TestPoint")
+		(at 69.85 138.43 0)
+		(unit 1)
+		(exclude_from_sim no)
+		(in_bom yes)
+		(on_board yes)
+		(dnp no)
+		(property "Reference" "TP6"
+			(at 68.072 133.35 0)
+			(effects
+				(font
+					(size 1.27 1.27)
+				)
+				(justify left)
+			)
+		)
+		(property "Value" "GPIO Breakout P0.24"
+			(at 64.516 130.556 0)
+			(effects
+				(font
+					(size 1.27 1.27)
+				)
+				(justify left)
+			)
+		)
+		(property "Footprint" "TestPoint:TestPoint_Pad_D1.0mm"
+			(at 74.93 138.43 0)
+			(effects
+				(font
+					(size 1.27 1.27)
+				)
+				(hide yes)
+			)
+		)
+		(property "Datasheet" "~"
+			(at 74.93 138.43 0)
+			(effects
+				(font
+					(size 1.27 1.27)
+				)
+				(hide yes)
+			)
+		)
+		(property "Description" "test point"
+			(at 69.85 138.43 0)
+			(effects
+				(font
+					(size 1.27 1.27)
+				)
+				(hide yes)
+			)
+		)
+		(pin "1"
+		)
+		(instances
+			(project "mic_patch_v1"
+				(path "/5448a297-4261-40a5-8009-47199bfe22cb/1e8f7a85-c9d9-4dea-908a-5a79456d7ca4"
+					(reference "TP6")
+					(unit 1)
+				)

Commit message: corrected missing part numbers + inconsistencies
Parts:
- R11, R13: value R_00002 -> R_00003
Changed lines of the file:
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@@
 			)
 		)
-		(property "Value" "R_00002"
+		(property "Value" "R_00003"
 			(at 50.8 133.3499 0)
 			(effects
@@
 			)
 		)
-		(property "Value" "R_00002"
+		(property "Value" "R_00003"
 			(at 50.8 165.0999 0)
 			(effects
